Commit message: feat: added base_link chassis to the robot urdf with one leg

File: quad_description/models/quad/monoped.xacro (robot description, xacro)
@@ -5,5 +5,5 @@
 *  Filename:			    quad.xacro
 *  Created:				    22/12/2023
-*  Last Modified:	    29/01/2024
+*  Last Modified:	    27/01/2024
 *  Author:				    Archit Jain
 *
@@ -54,29 +54,6 @@
     <child link="base_link" />
   </joint>
-  <!-- ********************** ROBOT BASELINK *********************************  -->
+  <!-- ********************** ROBOT BASE *********************************  -->
   <link name="base_link">
-    <visual>
-      <origin xyz="0 0 0" rpy="0 0 0"/>
-      <geometry>
-        <mesh filename="file://$(find quad_description)/meshes/base_link.obj" scale=".001 .001 .001"/>
-      </geometry>
-    </visual>
-    <collision>
-      <origin xyz="0 0 0" rpy="0 0 0"/>
-      <geometry>
-        <mesh filename="file://$(find quad_description)/meshes/base_link.obj" scale=".001 .001 .001"/>
-      </geometry>
-    </collision>
-    <xacro:box_inertia m="0.050" w="0.030" d="0.730" h="0.440">
-      <origin xyz="0 -0.015 0" rpy="1.571428571 0 1.571428571"/>
-    </xacro:box_inertia>
-  </link>
-  <joint name="hip_joint" type="fixed">
-    <origin xyz="0.300 -0.090 0.165" rpy="0 0 0"/>
-    <parent link="base_link"/>
-    <child link="hip_link" />
-  </joint>
-  <!-- ********************** HIP LINK *********************************  -->
-  <link name="hip_link">
     <visual>
       <origin xyz="0 0 0" rpy="0 0 0"/>
@@ -97,5 +74,5 @@
   <joint name="thigh_joint" type="revolute">
     <origin xyz="0 0 0" rpy="0 0 0"/>
-    <parent link="hip_link"/>
+    <parent link="base_link"/>
     <child link="thigh_link" />
     <axis xyz="0 0 1" />

File: quad_description/models/quad/monoped_gazebo.xacro (robot description, xacro)
@@ -3,8 +3,8 @@
 *****************************************************************************************
 *
-*  Filename:			    quad.gazebo
-*  Created:				    22/12/2023
-*  Last Modified:	    29/01/2024
-*  Author:				    Archit Jain
+*  Filename:			quad.gazebo
+*  Created:				22/12/2023
+*  Last Modified:	22/12/2023
+*  Author:				Archit Jain
 *
 *****************************************************************************************
@@ -14,7 +14,4 @@
   <xacro:property name="joint_limit" value="2.00712863979"/>    <!-- 115 degree -->
   <gazebo reference="base_link">
-    <material>Gazebo/Orange</material>
-  </gazebo>
-  <gazebo reference="hip_link">
     <material>Gazebo/Black</material>
   </gazebo>
