Commit message: fix: update in leg links friction values of mu1 and mu2

File: quad_description/models/quad/quad_gazebo.xacro (robot description, xacro)
@@ -5,5 +5,5 @@
 *  Filename:			    quad_gazebo.xacro
 *  Created:				    22/12/2023
-*  Last Modified:	    31/01/2024
+*  Last Modified:	    01/02/2024
 *  Author:				    Archit Jain
 *
@@ -15,6 +15,6 @@
   <xacro:property name="kp" value="1000000.0"/>
   <xacro:property name="kd" value="1.0"/>
-  <xacro:property name="mu1" value="0.15"/>
-  <xacro:property name="mu2" value="0.15"/>
+  <xacro:property name="mu1" value="0.8"/>
+  <xacro:property name="mu2" value="0.8"/>
   <xacro:property name="max_vel" value="0.0"/>
   <xacro:property name="min_depth" value="0.001"/>
