Commit message: fix: adjusted revolute joint for leg link

File: quad_description/models/quad/quad.xacro (robot description, xacro)
@@ -13,9 +13,11 @@
   <!-- ****************** BASIC INERTIAL MACROS ***************************  -->
   <!-- Define intertial property macros  -->
-  <xacro:macro name="box_inertia" params="m w h d">
+  <xacro:macro name="box_inertia" params="m w h d *origin">
     <inertial>
-      <origin xyz="0 0 0" rpy="${pi/2} 0 ${pi/2}"/>
+      <xacro:insert_block name="origin"/>
       <mass value="${m}"/>
-      <inertia ixx="${(m/12) * (h*h + d*d)}" ixy="0.0" ixz="0.0" iyy="${(m/12) * (w*w + d*d)}" iyz="0.0" izz="${(m/12) * (w*w + h*h)}"/>
+      <inertia  ixx="${(m/12) * (h*h + d*d)}" ixy="0.0" ixz="0.0"
+                iyy="${(m/12) * (w*w + d*d)}" iyz="0.0"
+                izz="${(m/12) * (w*w + h*h)}"/>
     </inertial>
   </xacro:macro>
@@ -35,32 +37,85 @@
   <!-- ****************** ROBOT CONSTANTS *******************************  -->
   <!-- Define the size of the robot's main chassis in meters -->
-  <xacro:property name="base_width" value="0.125"/>
-  <xacro:property name="base_length" value="0.035"/>
-  <xacro:property name="base_height" value="0.035"/>
-  <xacro:property name="base_mass" value="0.2"/>
+  <xacro:property name="base_width" value="0.550"/>
+  <xacro:property name="base_length" value="0.325"/>
+  <xacro:property name="base_height" value="0.025"/>
+  <xacro:property name="base_mass" value="0.4"/>
   <!-- ****************** ROBOT BASE FOOTPRINT ***************************  -->
   <!-- Define the center of the main robot chassis projected on the ground -->
-  <link name="base_footprint"/>
+  <link name="world"/>
   <!-- The base footprint of the robot is located underneath the chassis -->
   <joint name="base_joint" type="fixed">
-    <parent link="base_footprint"/>
+    <origin xyz="0.5 0.5 0" rpy="0 0 0"/>
+    <parent link="world"/>
     <child link="base_link" />
-    <origin xyz="0.0 0.0 0.0" rpy="0 0 0"/>
   </joint>
   <!-- ********************** ROBOT BASE *********************************  -->
   <link name="base_link">
     <visual>
-      <origin xyz="0 0 0" rpy="0 0 0"/>
+      <origin xyz="0 0 0.2" rpy="0 0 0"/>
       <geometry>
-        <mesh filename="file://$(find quad_description)/meshes/quad_limb.obj" scale=".001 .001 .001"/>
+        <box size="${base_length} ${base_width} ${base_height}"/>
       </geometry>
     </visual>
     <collision>
-      <origin xyz="0.015 -0.065 0.015" rpy="0 0 0"/>
+      <origin xyz="0 0 0.2" rpy="0 0 0"/>
       <geometry>
         <box size="${base_length} ${base_width} ${base_height}"/>
       </geometry>
     </collision>
-    <xacro:box_inertia m="${base_mass}" w="${base_width}" d="${base_length}" h="${base_height}"/>
+    <xacro:box_inertia m="${base_mass}" w="${base_width}" d="${base_length}" h="${base_height}">
+      <origin xyz="0 0 0.2" rpy="1.57 0 1.57"/>
+    </xacro:box_inertia>
   </link>
+  <joint name="leg_joint" type="revolute">
+    <origin xyz="${(base_length/2) + 0.005} ${(base_width/2) - 0.1} 0.2" rpy="1.57 0 1.57"/>
+    <parent link="base_link"/>
+    <child link="leg" />
+    <axis xyz="0 0 1" />
+    <limit effort="1000.0" lower="-1.57" upper="1.57" velocity="0.5"/>
+  </joint>
+  <!-- ********************** LEG *********************************  -->
+  <link name="leg">
+    <visual>
+      <origin xyz="-0.010700 -0.086500 0" rpy="0 0 0"/>
+      <geometry>
+        <mesh filename="file://$(find quad_description)/meshes/quad_leg.obj" scale=".001 .001 .001"/>
+      </geometry>
+    </visual>
+    <collision>
+      <origin xyz="-0.010700 -0.086500 0" rpy="0 0 0"/>
+      <geometry>
+        <mesh filename="file://$(find quad_description)/meshes/quad_leg.obj" scale=".001 .001 .001"/>
+        <!-- <box size="0.04 0.065 0.2"/> -->
+      </geometry>
+    </collision>
+    <xacro:box_inertia m="0.08" w="0.033" d="0.075" h="0.16">
+      <origin xyz="0.003 -0.055 0.016" rpy="0 0 0"/>
+    </xacro:box_inertia>
+  </link>
+    <!-- <joint name="leg_joint" type="revolute">
+    <origin xyz="${(base_length/2) + 0.005} ${(base_width/2) - 0.1} 0.2" rpy="1.57 0 1.57"/>
+    <parent link="base_link"/>
+    <child link="leg" />
+    <axis xyz="0 0 1" />
+    <limit effort="1000.0" lower="-1.57" upper="1.57" velocity="0.5"/>
+  </joint> -->
+  <!-- ********************** LEG *********************************  -->
+  <!-- <link name="limb">
+    <visual>
+      <origin xyz="-0.010700 -0.086500 0" rpy="0 0 0"/>
+      <geometry>
+        <mesh filename="file://$(find quad_description)/meshes/quad_leg.obj" scale=".001 .001 .001"/>
+      </geometry>
+    </visual>
+    <collision>
+      <origin xyz="-0.010700 -0.086500 0" rpy="0 0 0"/>
+      <geometry>
+        <mesh filename="file://$(find quad_description)/meshes/quad_leg.obj" scale=".001 .001 .001"/>
+      </geometry>
+    </collision>
+    <xacro:box_inertia m="0.08" w="0.0325" d="0.075" h="0.16">
+      <origin xyz="-0.010700 -0.086500 0" rpy="0 0 0"/>
+    </xacro:box_inertia>
+  </link> -->
 </robot>

Commit message: fix: adjusted revolute joint for limb link

File: quad_description/models/quad/quad.xacro (robot description, xacro)
@@ -41,4 +41,5 @@
   <xacro:property name="base_height" value="0.025"/>
   <xacro:property name="base_mass" value="0.4"/>
+  <xacro:property name="quad_height" value="0.15"/>
   <!-- ****************** ROBOT BASE FOOTPRINT ***************************  -->
   <!-- Define the center of the main robot chassis projected on the ground -->
@@ -53,5 +54,5 @@
   <link name="base_link">
     <visual>
-      <origin xyz="0 0 0.2" rpy="0 0 0"/>
+      <origin xyz="0 0 ${quad_height}" rpy="0 0 0"/>
       <geometry>
         <box size="${base_length} ${base_width} ${base_height}"/>
@@ -59,5 +60,5 @@
     </visual>
     <collision>
-      <origin xyz="0 0 0.2" rpy="0 0 0"/>
+      <origin xyz="0 0 ${quad_height}" rpy="0 0 0"/>
       <geometry>
         <box size="${base_length} ${base_width} ${base_height}"/>
@@ -65,13 +66,13 @@
     </collision>
     <xacro:box_inertia m="${base_mass}" w="${base_width}" d="${base_length}" h="${base_height}">
-      <origin xyz="0 0 0.2" rpy="1.57 0 1.57"/>
+      <origin xyz="0 0 ${quad_height}" rpy="1.57 0 1.57"/>
     </xacro:box_inertia>
   </link>
   <joint name="leg_joint" type="revolute">
-    <origin xyz="${(base_length/2) + 0.005} ${(base_width/2) - 0.1} 0.2" rpy="1.57 0 1.57"/>
+    <origin xyz="${(base_length/2) + 0.005} ${(base_width/2) - 0.1} ${quad_height}" rpy="1.57 0 1.57"/>
     <parent link="base_link"/>
     <child link="leg" />
     <axis xyz="0 0 1" />
-    <limit effort="1000.0" lower="-1.57" upper="1.57" velocity="0.5"/>
+    <limit effort="10.0" lower="-1.57" upper="1.57" velocity="0.5"/>
   </joint>
   <!-- ********************** LEG *********************************  -->
@@ -90,32 +91,33 @@
       </geometry>
     </collision>
-    <xacro:box_inertia m="0.08" w="0.033" d="0.075" h="0.16">
+    <xacro:box_inertia m="0.1" w="0.033" d="0.075" h="0.16">
       <origin xyz="0.003 -0.055 0.016" rpy="0 0 0"/>
     </xacro:box_inertia>
   </link>
-    <!-- <joint name="leg_joint" type="revolute">
-    <origin xyz="${(base_length/2) + 0.005} ${(base_width/2) - 0.1} 0.2" rpy="1.57 0 1.57"/>
-    <parent link="base_link"/>
-    <child link="leg" />
+  <joint name="limb_joint" type="revolute">
+    <origin xyz="0 -0.1095 0" rpy="0 0 0"/>
+    <parent link="leg" />
+    <child link="limb" />
     <axis xyz="0 0 1" />
-    <limit effort="1000.0" lower="-1.57" upper="1.57" velocity="0.5"/>
-  </joint> -->
+    <limit effort="10.0" lower="-1.57" upper="1.57" velocity="0.5"/>
+    <!-- <dynamics damping="1.0" /> -->
+  </joint>
   <!-- ********************** LEG *********************************  -->
-  <!-- <link name="limb">
+  <link name="limb">
     <visual>
-      <origin xyz="-0.010700 -0.086500 0" rpy="0 0 0"/>
+      <origin xyz="-0.01 0.023 0" rpy="0 0 0"/>
       <geometry>
-        <mesh filename="file://$(find quad_description)/meshes/quad_leg.obj" scale=".001 .001 .001"/>
+        <mesh filename="file://$(find quad_description)/meshes/quad_limb.obj" scale=".001 .001 .001"/>
       </geometry>
     </visual>
     <collision>
-      <origin xyz="-0.010700 -0.086500 0" rpy="0 0 0"/>
+      <origin xyz="-0.01 0.023 0" rpy="0 0 0"/>
       <geometry>
-        <mesh filename="file://$(find quad_description)/meshes/quad_leg.obj" scale=".001 .001 .001"/>
+        <mesh filename="file://$(find quad_description)/meshes/quad_limb.obj" scale=".001 .001 .001"/>
       </geometry>
     </collision>
-    <xacro:box_inertia m="0.08" w="0.0325" d="0.075" h="0.16">
-      <origin xyz="-0.010700 -0.086500 0" rpy="0 0 0"/>
+    <xacro:box_inertia m="0.08" w="0.0375" d="0.04375" h="0.13">
+      <origin xyz="0.0025 -0.04 0.015" rpy="0 0 0"/>
     </xacro:box_inertia>
-  </link> -->
+  </link>
 </robot>

Commit message: feat: added new design and urdf with base and thigh links

File: quad_description/models/quad/quad.xacro (robot description, xacro)
@@ -42,5 +42,5 @@
   <xacro:property name="base_height" value="0.025"/>
   <xacro:property name="base_mass" value="0.4"/>
-  <xacro:property name="quad_height" value="0.15"/>
+  <xacro:property name="quad_height" value="0.3"/>
   <!-- ****************** ROBOT BASE FOOTPRINT ***************************  -->
   <!-- Define the center of the main robot chassis projected on the ground -->
@@ -48,5 +48,5 @@
   <!-- The base footprint of the robot is located underneath the chassis -->
   <joint name="base_joint" type="fixed">
-    <origin xyz="0.5 0.5 0" rpy="0 0 0"/>
+    <origin xyz="0 0 ${quad_height}" rpy="1.571428571 0 0"/>
     <parent link="world"/>
     <child link="base_link" />
@@ -55,69 +55,41 @@
   <link name="base_link">
     <visual>
-      <origin xyz="0 0 ${quad_height}" rpy="0 0 0"/>
+      <origin xyz="0 0 0" rpy="0 0 0"/>
       <geometry>
-        <box size="${base_length} ${base_width} ${base_height}"/>
+        <mesh filename="file://$(find quad_description)/meshes/base.obj" scale=".001 .001 .001"/>
       </geometry>
     </visual>
     <collision>
-      <origin xyz="0 0 ${quad_height}" rpy="0 0 0"/>
+      <origin xyz="0 0 0" rpy="0 0 0"/>
       <geometry>
-        <box size="${base_length} ${base_width} ${base_height}"/>
+        <mesh filename="file://$(find quad_description)/meshes/base.obj" scale=".001 .001 .001"/>
       </geometry>
     </collision>
-    <xacro:box_inertia m="${base_mass}" w="${base_width}" d="${base_length}" h="${base_height}">
-      <origin xyz="0 0 ${quad_height}" rpy="1.57 0 1.57"/>
+    <xacro:box_inertia m="0.02" w="0.060" d="0.110" h="0.110">
+      <origin xyz="0 0.030 0" rpy="1.571428571 0 0"/>
     </xacro:box_inertia>
   </link>
-  <joint name="leg_joint" type="revolute">
-    <origin xyz="${(base_length/2) + 0.005} ${(base_width/2) - 0.1} ${quad_height}" rpy="1.57 0 1.57"/>
+  <joint name="thigh_joint" type="revolute">
+    <origin xyz="0 0 0" rpy="0 0 0"/>
     <parent link="base_link"/>
-    <child link="leg" />
-    <axis xyz="0 0 1" />
-    <limit effort="10.0" lower="-1.57" upper="1.57" velocity="0.5"/>
+    <child link="thigh_link" />
+    <axis xyz="0 1 0" />
+    <limit effort="200.0" lower="-1.571428571" upper="1.571428571" velocity="1.0"/>
   </joint>
-  <!-- ********************** LEG *********************************  -->
-  <link name="leg">
+  <link name="thigh_link">
     <visual>
-      <origin xyz="-0.010700 -0.086500 0" rpy="0 0 0"/>
+      <origin xyz="0 0 0" rpy="0 0 0"/>
       <geometry>
-        <mesh filename="file://$(find quad_description)/meshes/quad_leg.obj" scale=".001 .001 .001"/>
+        <mesh filename="file://$(find quad_description)/meshes/thigh.obj" scale=".001 .001 .001"/>
       </geometry>
     </visual>
     <collision>
-      <origin xyz="-0.010700 -0.086500 0" rpy="0 0 0"/>
+      <origin xyz="0 0 0" rpy="0 0 0"/>
       <geometry>
-        <mesh filename="file://$(find quad_description)/meshes/quad_leg.obj" scale=".001 .001 .001"/>
-        <!-- <box size="0.04 0.065 0.2"/> -->
+        <mesh filename="file://$(find quad_description)/meshes/thigh.obj" scale=".001 .001 .001"/>
       </geometry>
     </collision>
-    <xacro:box_inertia m="0.1" w="0.033" d="0.075" h="0.16">
-      <origin xyz="0.003 -0.055 0.016" rpy="0 0 0"/>
-    </xacro:box_inertia>
-  </link>
-  <joint name="limb_joint" type="revolute">
-    <origin xyz="0 -0.1095 0" rpy="0 0 0"/>
-    <parent link="leg" />
-    <child link="limb" />
-    <axis xyz="0 0 1" />
-    <limit effort="10.0" lower="-1.57" upper="1.57" velocity="0.5"/>
-    <!-- <dynamics damping="1.0" /> -->
-  </joint>
-  <!-- ********************** LEG *********************************  -->
-  <link name="limb">
-    <visual>
-      <origin xyz="-0.01 0.023 0" rpy="0 0 0"/>
-      <geometry>
-        <mesh filename="file://$(find quad_description)/meshes/quad_limb.obj" scale=".001 .001 .001"/>
-      </geometry>
-    </visual>
-    <collision>
-      <origin xyz="-0.01 0.023 0" rpy="0 0 0"/>
-      <geometry>
-        <mesh filename="file://$(find quad_description)/meshes/quad_limb.obj" scale=".001 .001 .001"/>
-      </geometry>
-    </collision>
-    <xacro:box_inertia m="0.08" w="0.0375" d="0.04375" h="0.13">
-      <origin xyz="0.0025 -0.04 0.015" rpy="0 0 0"/>
+    <xacro:box_inertia m="0.015" w="0.050" d="0.270" h="0.110">
+      <origin xyz="0 -0.110 0" rpy="1.571428571 0 0"/>
     </xacro:box_inertia>
   </link>

Commit message: feat: added leg link and joint

File: quad_description/models/quad/quad.xacro (robot description, xacro)
@@ -11,4 +11,5 @@
 -->
 <robot name="quad" xmlns:xacro="http://www.ros.org/wiki/xacro">
+  <!-- ****************** INCLUDE OTHER MACROS ***************************  -->
   <xacro:include filename="$(find quad_description)/models/quad/quad_gazebo.xacro" />
   <!-- ****************** BASIC INERTIAL MACROS ***************************  -->
@@ -42,5 +43,5 @@
   <xacro:property name="base_height" value="0.025"/>
   <xacro:property name="base_mass" value="0.4"/>
-  <xacro:property name="quad_height" value="0.3"/>
+  <xacro:property name="quad_height" value="0.5"/>
   <!-- ****************** ROBOT BASE FOOTPRINT ***************************  -->
   <!-- Define the center of the main robot chassis projected on the ground -->
@@ -77,4 +78,5 @@
     <limit effort="200.0" lower="-1.571428571" upper="1.571428571" velocity="1.0"/>
   </joint>
+  <!-- ********************** THIGH LINK *********************************  -->
   <link name="thigh_link">
     <visual>
@@ -94,3 +96,28 @@
     </xacro:box_inertia>
   </link>
+  <joint name="leg_joint" type="revolute">
+    <origin xyz="0 -0.220 0" rpy="0 0 0"/>
+    <parent link="thigh_link"/>
+    <child link="leg_link" />
+    <axis xyz="0 1 0" />
+    <limit effort="200.0" lower="-1.571428571" upper="1.571428571" velocity="1.0"/>
+  </joint>
+  <!-- ********************** LEG LINK *********************************  -->
+  <link name="leg_link">
+    <visual>
+      <origin xyz="0 0 0" rpy="0 0 0"/>
+      <geometry>
+        <mesh filename="file://$(find quad_description)/meshes/leg.obj" scale=".001 .001 .001"/>
+      </geometry>
+    </visual>
+    <collision>
+      <origin xyz="0 0 0" rpy="0 0 0"/>
+      <geometry>
+        <mesh filename="file://$(find quad_description)/meshes/leg.obj" scale=".001 .001 .001"/>
+      </geometry>
+    </collision>
+    <xacro:box_inertia m="0.0125" w="0.050" d="0.200" h="0.060">
+      <origin xyz="0 -0.075 0" rpy="1.571428571 0 0"/>
+    </xacro:box_inertia>
+  </link>
 </robot>

File: quad_description/models/quad/quad_gazebo.xacro (robot description, xacro)
@@ -15,8 +15,8 @@
     <material>Gazebo/Black</material>
   </gazebo>
-  <gazebo reference="leg">
+  <gazebo reference="thigh_link">
     <material>Gazebo/Orange</material>
   </gazebo>
-  <gazebo reference="limb">
+  <gazebo reference="leg_link">
     <material>Gazebo/Black</material>
   </gazebo>

Commit message: fix: revolute joint axis

File: quad_description/models/quad/quad.xacro (robot description, xacro)
@@ -75,5 +75,5 @@
     <parent link="base_link"/>
     <child link="thigh_link" />
-    <axis xyz="0 1 0" />
+    <axis xyz="0 0 1" />
     <limit effort="200.0" lower="-1.571428571" upper="1.571428571" velocity="1.0"/>
   </joint>
@@ -100,5 +100,5 @@
     <parent link="thigh_link"/>
     <child link="leg_link" />
-    <axis xyz="0 1 0" />
+    <axis xyz="0 0 1" />
     <limit effort="200.0" lower="-1.571428571" upper="1.571428571" velocity="1.0"/>
   </joint>

Commit message: fix: added friction, transmission and updated ros2_control tags

File: quad_description/models/quad/quad.xacro (robot description, xacro)
@@ -43,12 +43,12 @@
   <xacro:property name="base_height" value="0.025"/>
   <xacro:property name="base_mass" value="0.4"/>
-  <xacro:property name="quad_height" value="0.5"/>
+  <xacro:property name="quad_height" value="1.0"/>
   <!-- ****************** ROBOT BASE FOOTPRINT ***************************  -->
   <!-- Define the center of the main robot chassis projected on the ground -->
-  <link name="world"/>
+  <link name="base_footprint" />
   <!-- The base footprint of the robot is located underneath the chassis -->
   <joint name="base_joint" type="fixed">
     <origin xyz="0 0 ${quad_height}" rpy="1.571428571 0 0"/>
-    <parent link="world"/>
+    <parent link="base_footprint"/>
     <child link="base_link" />
   </joint>
@@ -76,5 +76,6 @@
     <child link="thigh_link" />
     <axis xyz="0 0 1" />
-    <limit effort="200.0" lower="-1.571428571" upper="1.571428571" velocity="1.0"/>
+    <limit effort="1.5" lower="-1.571428571" upper="1.571428571" velocity="1.0"/>
+    <dynamics damping="10.0" friction="1000.0" />
   </joint>
   <!-- ********************** THIGH LINK *********************************  -->
@@ -101,5 +102,6 @@
     <child link="leg_link" />
     <axis xyz="0 0 1" />
-    <limit effort="200.0" lower="-1.571428571" upper="1.571428571" velocity="1.0"/>
+    <limit effort="1.5" lower="-1.571428571" upper="1.571428571" velocity="1.0"/>
+    <dynamics damping="10.0" friction="1000.0" />
   </joint>
   <!-- ********************** LEG LINK *********************************  -->

File: quad_description/models/quad/quad_gazebo.xacro (robot description, xacro)
@@ -21,3 +21,96 @@
     <material>Gazebo/Black</material>
   </gazebo>
+  <gazebo reference="base_footprint">
+    <material>Gazebo/Black</material>
+  </gazebo>
+  <ros2_control name="GazeboSystem" type="system">
+    <hardware>
+      <plugin>gazebo_ros2_control/GazeboSystem</plugin>
+    </hardware>
+    <joint name="thigh_joint">
+      <command_interface name="position">
+        <param name="min">-1.571428571</param>
+        <param name="max">1.571428571</param>
+      </command_interface>
+      <state_interface name="position" />
+      <state_interface name="velocity" />
+      <state_interface name="effort" />
+    </joint>
+    <joint name="leg_joint">
+      <command_interface name="position">
+        <param name="min">-1.571428571</param>
+        <param name="max">1.571428571</param>
+      </command_interface>
+      <state_interface name="position" />
+      <state_interface name="velocity" />
+      <state_interface name="effort" />
+    </joint>
+  </ros2_control>
+  <transmission name="trans_thigh">
+    <type>transmission_interface/SimpleTransmission</type>
+    <joint name="thigh_joint">
+      <hardwareInterface>hardware_interface/EffortJointInterface</hardwareInterface>
+    </joint>
+    <actuator name="motor_thigh">
+      <hardwareInterface>hardware_interface/EffortJointInterface</hardwareInterface>
+      <mechanicalReduction>5</mechanicalReduction>
+    </actuator>
+  </transmission>
+  <transmission name="trans_leg">
+    <type>transmission_interface/SimpleTransmission</type>
+    <joint name="leg_joint">
+      <hardwareInterface>hardware_interface/EffortJointInterface</hardwareInterface>
+    </joint>
+    <actuator name="motor_leg">
+      <hardwareInterface>hardware_interface/EffortJointInterface</hardwareInterface>
+      <mechanicalReduction>5</mechanicalReduction>
+    </actuator>
+  </transmission>
+  <gazebo>
+    <plugin filename="libgazebo_ros2_control.so" name="gazebo_ros2_control">
+      <parameters>$(find quad_description)/config/quad_controllers.yaml</parameters>
+    </plugin>
+  </gazebo>
+  <gazebo reference="thigh_link">
+    <collision>
+      <surface>
+        <friction>
+          <ode>
+            <mu>1</mu>
+            <mu2>100</mu2>
+            <slip1>100.1</slip1>
+            <slip2>100.1</slip2>
+          </ode>
+        </friction>
+        <contact>
+          <ode>
+            <kp>1000000.0</kp>
+            <kd>100.0</kd>
+            <min_depth>0.001</min_depth>
+          </ode>
+        </contact>
+      </surface>
+    </collision>
+  </gazebo>
+  <gazebo reference="leg_link">
+    <collision>
+      <surface>
+        <friction>
+          <ode>
+            <mu>1</mu>
+            <mu2>100</mu2>
+            <slip1>100.1</slip1>
+            <slip2>100.1</slip2>
+          </ode>
+        </friction>
+        <contact>
+          <ode>
+            <kp>1000000.0</kp>
+            <kd>100.0</kd>
+            <min_depth>0.001</min_depth>
+          </ode>
+        </contact>
+      </surface>
+    </collision>
+  </gazebo>
 </robot>
