Commit message: feat: added joint limit dynamic variable of 115 deg

File: quad_description/models/quad/quad.xacro (robot description, xacro)
@@ -44,4 +44,5 @@
   <xacro:property name="base_mass" value="0.4"/>
   <xacro:property name="quad_height" value="1.0"/>
+  <xacro:property name="joint_limit" value="2.00712863979"/>      <!-- 115 degree -->
   <!-- ****************** ROBOT BASE FOOTPRINT ***************************  -->
   <!-- Define the center of the main robot chassis projected on the ground -->
@@ -76,5 +77,5 @@
     <child link="thigh_link" />
     <axis xyz="0 0 1" />
-    <limit effort="1.5" lower="-1.571428571" upper="1.571428571" velocity="1.0"/>
+    <limit effort="1.5" lower="-${joint_limit}" upper="${joint_limit}" velocity="1.0"/>
     <dynamics damping="10.0" friction="1000.0" />
   </joint>
@@ -102,5 +103,5 @@
     <child link="leg_link" />
     <axis xyz="0 0 1" />
-    <limit effort="1.5" lower="-1.571428571" upper="1.571428571" velocity="1.0"/>
+    <limit effort="1.5" lower="-${joint_limit}" upper="${joint_limit}" velocity="1.0"/>
     <dynamics damping="10.0" friction="1000.0" />
   </joint>

File: quad_description/models/quad/quad_gazebo.xacro (robot description, xacro)
@@ -12,4 +12,5 @@
 <robot name="quad"
   xmlns:xacro="http://www.ros.org/wiki/xacro">
+  <xacro:property name="joint_limit" value="2.00712863979"/>    <!-- 115 degree -->
   <gazebo reference="base_link">
     <material>Gazebo/Black</material>
@@ -30,6 +31,6 @@
     <joint name="thigh_joint">
       <command_interface name="position">
-        <param name="min">-1.571428571</param>
-        <param name="max">1.571428571</param>
+        <param name="min">-${joint_limit}</param>
+        <param name="max">${joint_limit}</param>
       </command_interface>
       <state_interface name="position" />
@@ -39,6 +40,6 @@
     <joint name="leg_joint">
       <command_interface name="position">
-        <param name="min">-1.571428571</param>
-        <param name="max">1.571428571</param>
+        <param name="min">-${joint_limit}</param>
+        <param name="max">${joint_limit}</param>
       </command_interface>
       <state_interface name="position" />

Commit message: fix: update in link length

File: quad_description/models/quad/quad.xacro (robot description, xacro)
@@ -3,8 +3,8 @@
 *****************************************************************************************
 *
-*  Filename:			quad.xacro
-*  Created:				22/12/2023
-*  Last Modified:	22/12/2023
-*  Author:				Archit Jain
+*  Filename:			    quad.xacro
+*  Created:				    22/12/2023
+*  Last Modified:	    27/01/2024
+*  Author:				    Archit Jain
 *
 *****************************************************************************************
@@ -120,6 +120,6 @@
       </geometry>
     </collision>
-    <xacro:box_inertia m="0.0125" w="0.050" d="0.200" h="0.060">
-      <origin xyz="0 -0.075 0" rpy="1.571428571 0 0"/>
+    <xacro:box_inertia m="0.0125" w="0.050" d="0.230" h="0.060">
+      <origin xyz="0 -0.090 0" rpy="1.571428571 0 0"/>
     </xacro:box_inertia>
   </link>

Commit message: fix: update in link length to equalize both links

File: quad_description/models/quad/quad.xacro (robot description, xacro)
@@ -120,6 +120,6 @@
       </geometry>
     </collision>
-    <xacro:box_inertia m="0.0125" w="0.050" d="0.230" h="0.060">
-      <origin xyz="0 -0.090 0" rpy="1.571428571 0 0"/>
+    <xacro:box_inertia m="0.0125" w="0.050" d="0.245" h="0.060">
+      <origin xyz="0 -0.0975 0" rpy="1.571428571 0 0"/>
     </xacro:box_inertia>
   </link>

Commit message: feat: created macros of each links and organized properly

File: quad_description/models/quad/quad.xacro (robot description, xacro)
@@ -13,4 +13,7 @@
   <!-- ****************** INCLUDE OTHER MACROS ***************************  -->
   <xacro:include filename="$(find quad_description)/models/quad/quad_gazebo.xacro" />
+  <xacro:include filename="$(find quad_description)/models/quad/quad_macros.xacro" />
+  <xacro:include filename="$(find quad_description)/models/quad/quad_ros2_control.xacro" />
+  <xacro:include filename="$(find quad_description)/models/quad/quad_transmission.xacro" />
   <!-- ****************** BASIC INERTIAL MACROS ***************************  -->
   <!-- Define intertial property macros  -->
@@ -48,102 +51,38 @@
   <!-- Define the center of the main robot chassis projected on the ground -->
   <link name="base_footprint" />
-  <!-- The base footprint of the robot is located underneath the chassis -->
-  <joint name="base_joint" type="fixed">
-    <origin xyz="0 0 ${quad_height}" rpy="1.571428571 0 0"/>
-    <parent link="base_footprint"/>
-    <child link="base_link" />
-  </joint>
+  <xacro:fixed_joint
+    joint_name="base_joint"
+    parent_link="base_footprint"
+    child_link="base_link"
+    pos_x="0" pos_y="0" pos_z="${quad_height}"
+    rot_x="1.571428571" rot_y="0" rot_z="0"/>
   <!-- ********************** ROBOT BASELINK *********************************  -->
-  <link name="base_link">
-    <visual>
-      <origin xyz="0 0 0" rpy="0 0 0"/>
-      <geometry>
-        <mesh filename="file://$(find quad_description)/meshes/base_link.obj" scale=".001 .001 .001"/>
-      </geometry>
-    </visual>
-    <collision>
-      <origin xyz="0 0 0" rpy="0 0 0"/>
-      <geometry>
-        <mesh filename="file://$(find quad_description)/meshes/base_link.obj" scale=".001 .001 .001"/>
-      </geometry>
-    </collision>
-    <xacro:box_inertia m="0.050" w="0.030" d="0.730" h="0.440">
-      <origin xyz="0 -0.015 0" rpy="1.571428571 0 1.571428571"/>
-    </xacro:box_inertia>
-  </link>
-  <joint name="hip_joint" type="fixed">
-    <origin xyz="0.300 -0.090 0.165" rpy="0 0 0"/>
-    <parent link="base_link"/>
-    <child link="hip_link" />
-  </joint>
-  <!-- ********************** HIP LINK *********************************  -->
-  <link name="hip_link">
-    <visual>
-      <origin xyz="0 0 0" rpy="0 0 0"/>
-      <geometry>
-        <mesh filename="file://$(find quad_description)/meshes/hip.obj" scale=".001 .001 .001"/>
-      </geometry>
-    </visual>
-    <collision>
-      <origin xyz="0 0 0" rpy="0 0 0"/>
-      <geometry>
-        <mesh filename="file://$(find quad_description)/meshes/hip.obj" scale=".001 .001 .001"/>
-      </geometry>
-    </collision>
-    <xacro:box_inertia m="0.02" w="0.060" d="0.110" h="0.110">
-      <origin xyz="0 0.030 0" rpy="1.571428571 0 0"/>
-    </xacro:box_inertia>
-  </link>
-  <joint name="thigh_joint" type="revolute">
-    <origin xyz="0 0 0" rpy="0 0 0"/>
-    <parent link="hip_link"/>
-    <child link="thigh_link" />
-    <axis xyz="0 0 1" />
-    <limit effort="1.5" lower="-${joint_limit}" upper="${joint_limit}" velocity="1.0"/>
-    <dynamics damping="10.0" friction="1000.0" />
-  </joint>
-  <!-- ********************** THIGH LINK *********************************  -->
-  <link name="thigh_link">
-    <visual>
-      <origin xyz="0 0 0" rpy="0 0 0"/>
-      <geometry>
-        <mesh filename="file://$(find quad_description)/meshes/thigh.obj" scale=".001 .001 .001"/>
-      </geometry>
-    </visual>
-    <collision>
-      <origin xyz="0 0 0" rpy="0 0 0"/>
-      <geometry>
-        <mesh filename="file://$(find quad_description)/meshes/thigh.obj" scale=".001 .001 .001"/>
-      </geometry>
-    </collision>
-    <xacro:box_inertia m="0.015" w="0.050" d="0.270" h="0.110">
-      <origin xyz="0 -0.110 0" rpy="1.571428571 0 0"/>
-    </xacro:box_inertia>
-  </link>
-  <joint name="leg_joint" type="revolute">
-    <origin xyz="0 -0.220 0" rpy="0 0 0"/>
-    <parent link="thigh_link"/>
-    <child link="leg_link" />
-    <axis xyz="0 0 1" />
-    <limit effort="1.5" lower="-${joint_limit}" upper="${joint_limit}" velocity="1.0"/>
-    <dynamics damping="10.0" friction="1000.0" />
-  </joint>
-  <!-- ********************** LEG LINK *********************************  -->
-  <link name="leg_link">
-    <visual>
-      <origin xyz="0 0 0" rpy="0 0 0"/>
-      <geometry>
-        <mesh filename="file://$(find quad_description)/meshes/leg.obj" scale=".001 .001 .001"/>
-      </geometry>
-    </visual>
-    <collision>
-      <origin xyz="0 0 0" rpy="0 0 0"/>
-      <geometry>
-        <mesh filename="file://$(find quad_description)/meshes/leg.obj" scale=".001 .001 .001"/>
-      </geometry>
-    </collision>
-    <xacro:box_inertia m="0.0125" w="0.050" d="0.245" h="0.060">
-      <origin xyz="0 -0.0975 0" rpy="1.571428571 0 0"/>
-    </xacro:box_inertia>
-  </link>
+  <xacro:base_link link_name="base_link"/>
+  <xacro:fixed_joint
+    joint_name="hip_joint_fr"
+    parent_link="base_link"
+    child_link="hip_link_fr"
+    pos_x="0.300" pos_y="-0.090" pos_z="0.165"
+    rot_x="0" rot_y="0" rot_z="0"/>
+  <xacro:hip_link link_name="hip_link_fr"/>
+  <xacro:revolute_joint
+    joint_name="thigh_joint_fr"
+    parent_link="hip_link_fr"
+    child_link="thigh_link_fr"
+    axis_x="0" axis_y="0" axis_z="1"
+    pos_x="0" pos_y="0" pos_z="0"
+    rot_x="0" rot_y="0" rot_z="0"
+    effort="1.5" joint_limit_l="-${joint_limit}" joint_limit_u="${joint_limit}" velocity="1.0"
+    damping="10.0" friction="1000.0" />
+  <xacro:thigh_link link_name="thigh_link_fr"/>
+  <xacro:revolute_joint
+    joint_name="leg_joint_fr"
+    parent_link="thigh_link_fr"
+    child_link="leg_link_fr"
+    axis_x="0" axis_y="0" axis_z="1"
+    pos_x="0" pos_y="-0.220" pos_z="0"
+    rot_x="0" rot_y="0" rot_z="0"
+    effort="1.5" joint_limit_l="-${joint_limit}" joint_limit_u="${joint_limit}" velocity="1.0"
+    damping="10.0" friction="1000.0" />
+  <xacro:leg_link link_name="leg_link_fr"/>
 </robot>

File: quad_description/models/quad/quad_gazebo.xacro (robot description, xacro)
@@ -3,5 +3,5 @@
 *****************************************************************************************
 *
-*  Filename:			    quad.gazebo
+*  Filename:			    quad_gazebo.xacro
 *  Created:				    22/12/2023
 *  Last Modified:	    29/01/2024
@@ -16,11 +16,11 @@
     <material>Gazebo/Orange</material>
   </gazebo>
-  <gazebo reference="hip_link">
+  <gazebo reference="hip_link_fr">
     <material>Gazebo/Black</material>
   </gazebo>
-  <gazebo reference="thigh_link">
+  <gazebo reference="thigh_link_fr">
     <material>Gazebo/Orange</material>
   </gazebo>
-  <gazebo reference="leg_link">
+  <gazebo reference="leg_link_fr">
     <material>Gazebo/Black</material>
   </gazebo>
@@ -28,47 +28,4 @@
     <material>Gazebo/Black</material>
   </gazebo>
-  <ros2_control name="GazeboSystem" type="system">
-    <hardware>
-      <plugin>gazebo_ros2_control/GazeboSystem</plugin>
-    </hardware>
-    <joint name="thigh_joint">
-      <command_interface name="position">
-        <param name="min">-${joint_limit}</param>
-        <param name="max">${joint_limit}</param>
-      </command_interface>
-      <state_interface name="position" />
-      <state_interface name="velocity" />
-      <state_interface name="effort" />
-    </joint>
-    <joint name="leg_joint">
-      <command_interface name="position">
-        <param name="min">-${joint_limit}</param>
-        <param name="max">${joint_limit}</param>
-      </command_interface>
-      <state_interface name="position" />
-      <state_interface name="velocity" />
-      <state_interface name="effort" />
-    </joint>
-  </ros2_control>
-  <transmission name="trans_thigh">
-    <type>transmission_interface/SimpleTransmission</type>
-    <joint name="thigh_joint">
-      <hardwareInterface>hardware_interface/EffortJointInterface</hardwareInterface>
-    </joint>
-    <actuator name="motor_thigh">
-      <hardwareInterface>hardware_interface/EffortJointInterface</hardwareInterface>
-      <mechanicalReduction>5</mechanicalReduction>
-    </actuator>
-  </transmission>
-  <transmission name="trans_leg">
-    <type>transmission_interface/SimpleTransmission</type>
-    <joint name="leg_joint">
-      <hardwareInterface>hardware_interface/EffortJointInterface</hardwareInterface>
-    </joint>
-    <actuator name="motor_leg">
-      <hardwareInterface>hardware_interface/EffortJointInterface</hardwareInterface>
-      <mechanicalReduction>5</mechanicalReduction>
-    </actuator>
-  </transmission>
   <gazebo>
     <plugin filename="libgazebo_ros2_control.so" name="gazebo_ros2_control">
@@ -76,5 +33,5 @@
     </plugin>
   </gazebo>
-  <gazebo reference="thigh_link">
+  <gazebo reference="thigh_link_fr">
     <collision>
       <surface>
@@ -97,5 +54,5 @@
     </collision>
   </gazebo>
-  <gazebo reference="leg_link">
+  <gazebo reference="leg_link_fr">
     <collision>
       <surface>

Commit message: feat: added front left links

File: quad_description/models/quad/quad.xacro (robot description, xacro)
@@ -59,4 +59,5 @@
   <!-- ********************** ROBOT BASELINK *********************************  -->
   <xacro:base_link link_name="base_link"/>
+  <!-- ********************** FRONT RIGHT LINKS *********************************  -->
   <xacro:fixed_joint
     joint_name="hip_joint_fr"
@@ -86,3 +87,31 @@
     damping="10.0" friction="1000.0" />
   <xacro:leg_link link_name="leg_link_fr"/>
+  <!-- ********************** FRONT LEFT LINKS *********************************  -->
+  <xacro:fixed_joint
+    joint_name="hip_joint_fl"
+    parent_link="base_link"
+    child_link="hip_link_fl"
+    pos_x="0.300" pos_y="-0.090" pos_z="-0.165"
+    rot_x="0" rot_y="0" rot_z="0"/>
+  <xacro:hip_link link_name="hip_link_fl"/>
+  <xacro:revolute_joint
+    joint_name="thigh_joint_fl"
+    parent_link="hip_link_fl"
+    child_link="thigh_link_fl"
+    axis_x="0" axis_y="0" axis_z="1"
+    pos_x="0" pos_y="0" pos_z="0"
+    rot_x="0" rot_y="0" rot_z="0"
+    effort="1.5" joint_limit_l="-${joint_limit}" joint_limit_u="${joint_limit}" velocity="1.0"
+    damping="10.0" friction="1000.0" />
+  <xacro:thigh_link link_name="thigh_link_fl"/>
+  <xacro:revolute_joint
+    joint_name="leg_joint_fl"
+    parent_link="thigh_link_fl"
+    child_link="leg_link_fl"
+    axis_x="0" axis_y="0" axis_z="1"
+    pos_x="0" pos_y="-0.220" pos_z="0"
+    rot_x="0" rot_y="0" rot_z="0"
+    effort="1.5" joint_limit_l="-${joint_limit}" joint_limit_u="${joint_limit}" velocity="1.0"
+    damping="10.0" friction="1000.0" />
+  <xacro:leg_link link_name="leg_link_fl"/>
 </robot>

File: quad_description/models/quad/quad_gazebo.xacro (robot description, xacro)
@@ -16,4 +16,7 @@
     <material>Gazebo/Orange</material>
   </gazebo>
+  <gazebo reference="base_footprint">
+    <material>Gazebo/Black</material>
+  </gazebo>
   <gazebo reference="hip_link_fr">
     <material>Gazebo/Black</material>
@@ -25,5 +28,11 @@
     <material>Gazebo/Black</material>
   </gazebo>
-  <gazebo reference="base_footprint">
+  <gazebo reference="hip_link_fl">
+    <material>Gazebo/Black</material>
+  </gazebo>
+  <gazebo reference="thigh_link_fl">
+    <material>Gazebo/Orange</material>
+  </gazebo>
+  <gazebo reference="leg_link_fl">
     <material>Gazebo/Black</material>
   </gazebo>
@@ -75,3 +84,45 @@
     </collision>
   </gazebo>
+  <gazebo reference="thigh_link_fl">
+    <collision>
+      <surface>
+        <friction>
+          <ode>
+            <mu>1</mu>
+            <mu2>100</mu2>
+            <slip1>100.1</slip1>
+            <slip2>100.1</slip2>
+          </ode>
+        </friction>
+        <contact>
+          <ode>
+            <kp>1000000.0</kp>
+            <kd>100.0</kd>
+            <min_depth>0.001</min_depth>
+          </ode>
+        </contact>
+      </surface>
+    </collision>
+  </gazebo>
+  <gazebo reference="leg_link_fl">
+    <collision>
+      <surface>
+        <friction>
+          <ode>
+            <mu>1</mu>
+            <mu2>100</mu2>
+            <slip1>100.1</slip1>
+            <slip2>100.1</slip2>
+          </ode>
+        </friction>
+        <contact>
+          <ode>
+            <kp>1000000.0</kp>
+            <kd>100.0</kd>
+            <min_depth>0.001</min_depth>
+          </ode>
+        </contact>
+      </surface>
+    </collision>
+  </gazebo>
 </robot>

File: quad_description/models/quad/quad_ros2_control.xacro (robot description, xacro)
@@ -16,4 +16,5 @@
       <plugin>gazebo_ros2_control/GazeboSystem</plugin>
     </hardware>
+    <!-- ********************** FRONT RIGHT JOINTS *********************************  -->
     <joint name="thigh_joint_fr">
       <command_interface name="position">
@@ -34,4 +35,23 @@
       <state_interface name="effort" />
     </joint>
+    <!-- ********************** FRONT LEFT JOINTS *********************************  -->
+    <joint name="thigh_joint_fl">
+      <command_interface name="position">
+        <param name="min">-${joint_limit}</param>
+        <param name="max">${joint_limit}</param>
+      </command_interface>
+      <state_interface name="position" />
+      <state_interface name="velocity" />
+      <state_interface name="effort" />
+    </joint>
+    <joint name="leg_joint_fl">
+      <command_interface name="position">
+        <param name="min">-${joint_limit}</param>
+        <param name="max">${joint_limit}</param>
+      </command_interface>
+      <state_interface name="position" />
+      <state_interface name="velocity" />
+      <state_interface name="effort" />
+    </joint>
   </ros2_control>
 </robot>

File: quad_description/models/quad/quad_transmission.xacro (robot description, xacro)
@@ -12,4 +12,5 @@
 <robot name="quad"
   xmlns:xacro="http://www.ros.org/wiki/xacro">
+  <!-- ********************** FRONT RIGHT JOINTS *********************************  -->
   <transmission name="trans_thigh_fr">
     <type>transmission_interface/SimpleTransmission</type>
@@ -32,3 +33,24 @@
     </actuator>
   </transmission>
+  <!-- ********************** FRONT LEFT JOINTS *********************************  -->
+  <transmission name="trans_thigh_fl">
+    <type>transmission_interface/SimpleTransmission</type>
+    <joint name="thigh_joint_fl">
+      <hardwareInterface>hardware_interface/EffortJointInterface</hardwareInterface>
+    </joint>
+    <actuator name="motor_thigh_fl">
+      <hardwareInterface>hardware_interface/EffortJointInterface</hardwareInterface>
+      <mechanicalReduction>5</mechanicalReduction>
+    </actuator>
+  </transmission>
+  <transmission name="trans_leg_fl">
+    <type>transmission_interface/SimpleTransmission</type>
+    <joint name="leg_joint_fl">
+      <hardwareInterface>hardware_interface/EffortJointInterface</hardwareInterface>
+    </joint>
+    <actuator name="motor_leg_fl">
+      <hardwareInterface>hardware_interface/EffortJointInterface</hardwareInterface>
+      <mechanicalReduction>5</mechanicalReduction>
+    </actuator>
+  </transmission>
 </robot>
