Commit message: feat: added rear left and right links

File: quad_description/models/quad/quad.xacro (robot description, xacro)
@@ -115,3 +115,59 @@
     damping="10.0" friction="1000.0" />
   <xacro:leg_link link_name="leg_link_fl"/>
+  <!-- ********************** REAR RIGHT LINKS *********************************  -->
+  <xacro:fixed_joint
+    joint_name="hip_joint_rr"
+    parent_link="base_link"
+    child_link="hip_link_rr"
+    pos_x="-0.300" pos_y="-0.090" pos_z="0.165"
+    rot_x="0" rot_y="0" rot_z="0"/>
+  <xacro:hip_link link_name="hip_link_rr"/>
+  <xacro:revolute_joint
+    joint_name="thigh_joint_rr"
+    parent_link="hip_link_rr"
+    child_link="thigh_link_rr"
+    axis_x="0" axis_y="0" axis_z="1"
+    pos_x="0" pos_y="0" pos_z="0"
+    rot_x="0" rot_y="0" rot_z="0"
+    effort="1.5" joint_limit_l="-${joint_limit}" joint_limit_u="${joint_limit}" velocity="1.0"
+    damping="10.0" friction="1000.0" />
+  <xacro:thigh_link link_name="thigh_link_rr"/>
+  <xacro:revolute_joint
+    joint_name="leg_joint_rr"
+    parent_link="thigh_link_rr"
+    child_link="leg_link_rr"
+    axis_x="0" axis_y="0" axis_z="1"
+    pos_x="0" pos_y="-0.220" pos_z="0"
+    rot_x="0" rot_y="0" rot_z="0"
+    effort="1.5" joint_limit_l="-${joint_limit}" joint_limit_u="${joint_limit}" velocity="1.0"
+    damping="10.0" friction="1000.0" />
+  <xacro:leg_link link_name="leg_link_rr"/>
+  <!-- ********************** REAR LEFT LINKS *********************************  -->
+  <xacro:fixed_joint
+    joint_name="hip_joint_rl"
+    parent_link="base_link"
+    child_link="hip_link_rl"
+    pos_x="-0.300" pos_y="-0.090" pos_z="-0.165"
+    rot_x="0" rot_y="0" rot_z="0"/>
+  <xacro:hip_link link_name="hip_link_rl"/>
+  <xacro:revolute_joint
+    joint_name="thigh_joint_rl"
+    parent_link="hip_link_rl"
+    child_link="thigh_link_rl"
+    axis_x="0" axis_y="0" axis_z="1"
+    pos_x="0" pos_y="0" pos_z="0"
+    rot_x="0" rot_y="0" rot_z="0"
+    effort="1.5" joint_limit_l="-${joint_limit}" joint_limit_u="${joint_limit}" velocity="1.0"
+    damping="10.0" friction="1000.0" />
+  <xacro:thigh_link link_name="thigh_link_rl"/>
+  <xacro:revolute_joint
+    joint_name="leg_joint_rl"
+    parent_link="thigh_link_rl"
+    child_link="leg_link_rl"
+    axis_x="0" axis_y="0" axis_z="1"
+    pos_x="0" pos_y="-0.220" pos_z="0"
+    rot_x="0" rot_y="0" rot_z="0"
+    effort="1.5" joint_limit_l="-${joint_limit}" joint_limit_u="${joint_limit}" velocity="1.0"
+    damping="10.0" friction="1000.0" />
+  <xacro:leg_link link_name="leg_link_rl"/>
 </robot>

File: quad_description/models/quad/quad_gazebo.xacro (robot description, xacro)
@@ -35,4 +35,22 @@
   </gazebo>
   <gazebo reference="leg_link_fl">
+    <material>Gazebo/Black</material>
+  </gazebo>
+  <gazebo reference="hip_link_rr">
+    <material>Gazebo/Black</material>
+  </gazebo>
+  <gazebo reference="thigh_link_rr">
+    <material>Gazebo/Orange</material>
+  </gazebo>
+  <gazebo reference="leg_link_rr">
+    <material>Gazebo/Black</material>
+  </gazebo>
+  <gazebo reference="hip_link_rl">
+    <material>Gazebo/Black</material>
+  </gazebo>
+  <gazebo reference="thigh_link_rl">
+    <material>Gazebo/Orange</material>
+  </gazebo>
+  <gazebo reference="leg_link_rl">
     <material>Gazebo/Black</material>
   </gazebo>

File: quad_description/models/quad/quad_ros2_control.xacro (robot description, xacro)
@@ -54,4 +54,42 @@
       <state_interface name="effort" />
     </joint>
+    <!-- ********************** REAR RIGHT JOINTS *********************************  -->
+    <joint name="thigh_joint_rr">
+      <command_interface name="position">
+        <param name="min">-${joint_limit}</param>
+        <param name="max">${joint_limit}</param>
+      </command_interface>
+      <state_interface name="position" />
+      <state_interface name="velocity" />
+      <state_interface name="effort" />
+    </joint>
+    <joint name="leg_joint_rr">
+      <command_interface name="position">
+        <param name="min">-${joint_limit}</param>
+        <param name="max">${joint_limit}</param>
+      </command_interface>
+      <state_interface name="position" />
+      <state_interface name="velocity" />
+      <state_interface name="effort" />
+    </joint>
+    <!-- ********************** REAR LEFT JOINTS *********************************  -->
+    <joint name="thigh_joint_rl">
+      <command_interface name="position">
+        <param name="min">-${joint_limit}</param>
+        <param name="max">${joint_limit}</param>
+      </command_interface>
+      <state_interface name="position" />
+      <state_interface name="velocity" />
+      <state_interface name="effort" />
+    </joint>
+    <joint name="leg_joint_rl">
+      <command_interface name="position">
+        <param name="min">-${joint_limit}</param>
+        <param name="max">${joint_limit}</param>
+      </command_interface>
+      <state_interface name="position" />
+      <state_interface name="velocity" />
+      <state_interface name="effort" />
+    </joint>
   </ros2_control>
 </robot>

File: quad_description/models/quad/quad_transmission.xacro (robot description, xacro)
@@ -54,3 +54,45 @@
     </actuator>
   </transmission>
+  <!-- ********************** REAR RIGHT JOINTS *********************************  -->
+  <transmission name="trans_thigh_rr">
+    <type>transmission_interface/SimpleTransmission</type>
+    <joint name="thigh_joint_rr">
+      <hardwareInterface>hardware_interface/EffortJointInterface</hardwareInterface>
+    </joint>
+    <actuator name="motor_thigh_rr">
+      <hardwareInterface>hardware_interface/EffortJointInterface</hardwareInterface>
+      <mechanicalReduction>5</mechanicalReduction>
+    </actuator>
+  </transmission>
+  <transmission name="trans_leg_rr">
+    <type>transmission_interface/SimpleTransmission</type>
+    <joint name="leg_joint_rr">
+      <hardwareInterface>hardware_interface/EffortJointInterface</hardwareInterface>
+    </joint>
+    <actuator name="motor_leg_rr">
+      <hardwareInterface>hardware_interface/EffortJointInterface</hardwareInterface>
+      <mechanicalReduction>5</mechanicalReduction>
+    </actuator>
+  </transmission>
+  <!-- ********************** REAR LEFT JOINTS *********************************  -->
+  <transmission name="trans_thigh_rl">
+    <type>transmission_interface/SimpleTransmission</type>
+    <joint name="thigh_joint_rl">
+      <hardwareInterface>hardware_interface/EffortJointInterface</hardwareInterface>
+    </joint>
+    <actuator name="motor_thigh_rl">
+      <hardwareInterface>hardware_interface/EffortJointInterface</hardwareInterface>
+      <mechanicalReduction>5</mechanicalReduction>
+    </actuator>
+  </transmission>
+  <transmission name="trans_leg_rl">
+    <type>transmission_interface/SimpleTransmission</type>
+    <joint name="leg_joint_rl">
+      <hardwareInterface>hardware_interface/EffortJointInterface</hardwareInterface>
+    </joint>
+    <actuator name="motor_leg_rl">
+      <hardwareInterface>hardware_interface/EffortJointInterface</hardwareInterface>
+      <mechanicalReduction>5</mechanicalReduction>
+    </actuator>
+  </transmission>
 </robot>

Commit message: fix: updated joint limit, removed friction, modified weight of  links

File: quad_description/models/quad/quad.xacro (robot description, xacro)
@@ -47,5 +47,5 @@
   <xacro:property name="base_mass" value="0.4"/>
   <xacro:property name="quad_height" value="1.0"/>
-  <xacro:property name="joint_limit" value="2.00712863979"/>      <!-- 115 degree -->
+  <xacro:property name="joint_limit" value="2.09439510239"/>      <!-- 120 degree -->
   <!-- ****************** ROBOT BASE FOOTPRINT ***************************  -->
   <!-- Define the center of the main robot chassis projected on the ground -->

File: quad_description/models/quad/quad_gazebo.xacro (robot description, xacro)
@@ -12,5 +12,5 @@
 <robot name="quad"
   xmlns:xacro="http://www.ros.org/wiki/xacro">
-  <xacro:property name="joint_limit" value="2.00712863979"/>    <!-- 115 degree -->
+  <xacro:property name="joint_limit" value="2.09439510239"/>      <!-- 120 degree -->
   <gazebo reference="base_link">
     <material>Gazebo/Orange</material>
@@ -60,87 +60,3 @@
     </plugin>
   </gazebo>
-  <gazebo reference="thigh_link_fr">
-    <collision>
-      <surface>
-        <friction>
-          <ode>
-            <mu>1</mu>
-            <mu2>100</mu2>
-            <slip1>100.1</slip1>
-            <slip2>100.1</slip2>
-          </ode>
-        </friction>
-        <contact>
-          <ode>
-            <kp>1000000.0</kp>
-            <kd>100.0</kd>
-            <min_depth>0.001</min_depth>
-          </ode>
-        </contact>
-      </surface>
-    </collision>
-  </gazebo>
-  <gazebo reference="leg_link_fr">
-    <collision>
-      <surface>
-        <friction>
-          <ode>
-            <mu>1</mu>
-            <mu2>100</mu2>
-            <slip1>100.1</slip1>
-            <slip2>100.1</slip2>
-          </ode>
-        </friction>
-        <contact>
-          <ode>
-            <kp>1000000.0</kp>
-            <kd>100.0</kd>
-            <min_depth>0.001</min_depth>
-          </ode>
-        </contact>
-      </surface>
-    </collision>
-  </gazebo>
-  <gazebo reference="thigh_link_fl">
-    <collision>
-      <surface>
-        <friction>
-          <ode>
-            <mu>1</mu>
-            <mu2>100</mu2>
-            <slip1>100.1</slip1>
-            <slip2>100.1</slip2>
-          </ode>
-        </friction>
-        <contact>
-          <ode>
-            <kp>1000000.0</kp>
-            <kd>100.0</kd>
-            <min_depth>0.001</min_depth>
-          </ode>
-        </contact>
-      </surface>
-    </collision>
-  </gazebo>
-  <gazebo reference="leg_link_fl">
-    <collision>
-      <surface>
-        <friction>
-          <ode>
-            <mu>1</mu>
-            <mu2>100</mu2>
-            <slip1>100.1</slip1>
-            <slip2>100.1</slip2>
-          </ode>
-        </friction>
-        <contact>
-          <ode>
-            <kp>1000000.0</kp>
-            <kd>100.0</kd>
-            <min_depth>0.001</min_depth>
-          </ode>
-        </contact>
-      </surface>
-    </collision>
-  </gazebo>
 </robot>

File: quad_description/models/quad/quad_macros.xacro (robot description, xacro)
@@ -26,5 +26,5 @@
         </geometry>
       </collision>
-      <xacro:box_inertia m="0.02" w="0.060" d="0.110" h="0.110">
+      <xacro:box_inertia m="0.020" w="0.060" d="0.110" h="0.110">
         <origin xyz="0 0.030 0" rpy="1.571428571 0 0"/>
       </xacro:box_inertia>
@@ -62,5 +62,5 @@
         </geometry>
       </collision>
-      <xacro:box_inertia m="0.050" w="0.030" d="0.730" h="0.440">
+      <xacro:box_inertia m="0.300" w="0.030" d="0.730" h="0.440">
         <origin xyz="0 -0.015 0" rpy="1.571428571 0 1.571428571"/>
       </xacro:box_inertia>
@@ -81,5 +81,5 @@
         </geometry>
       </collision>
-      <xacro:box_inertia m="0.015" w="0.050" d="0.270" h="0.110">
+      <xacro:box_inertia m="0.050" w="0.050" d="0.270" h="0.110">
         <origin xyz="0 -0.110 0" rpy="1.571428571 0 0"/>
       </xacro:box_inertia>
@@ -100,5 +100,5 @@
         </geometry>
       </collision>
-      <xacro:box_inertia m="0.0125" w="0.050" d="0.245" h="0.060">
+      <xacro:box_inertia m="0.050" w="0.050" d="0.245" h="0.060">
         <origin xyz="0 -0.0975 0" rpy="1.571428571 0 0"/>
       </xacro:box_inertia>

Commit message: fix: dynamic friction and damping variables

File: quad_description/models/quad/quad.xacro (robot description, xacro)
@@ -15,5 +15,5 @@
   <xacro:include filename="$(find quad_description)/models/quad/quad_macros.xacro" />
   <xacro:include filename="$(find quad_description)/models/quad/quad_ros2_control.xacro" />
-  <xacro:include filename="$(find quad_description)/models/quad/quad_transmission.xacro" />
+  <!-- <xacro:include filename="$(find quad_description)/models/quad/quad_transmission.xacro" /> -->
   <!-- ****************** BASIC INERTIAL MACROS ***************************  -->
   <!-- Define intertial property macros  -->
@@ -48,4 +48,6 @@
   <xacro:property name="quad_height" value="1.0"/>
   <xacro:property name="joint_limit" value="2.09439510239"/>      <!-- 120 degree -->
+  <xacro:property name="damping" value="0.5"/>
+  <xacro:property name="friction" value="0.15"/>         <!-- ABS=0.35 -->
   <!-- ****************** ROBOT BASE FOOTPRINT ***************************  -->
   <!-- Define the center of the main robot chassis projected on the ground -->
@@ -56,5 +58,5 @@
     child_link="base_link"
     pos_x="0" pos_y="0" pos_z="${quad_height}"
-    rot_x="1.571428571" rot_y="0" rot_z="0"/>
+    rot_x="1.571428571" rot_y="0.75" rot_z="0"/>      <!-- Originally set it to (90 0 0) -->
   <!-- ********************** ROBOT BASELINK *********************************  -->
   <xacro:base_link link_name="base_link"/>
@@ -74,6 +76,6 @@
     pos_x="0" pos_y="0" pos_z="0"
     rot_x="0" rot_y="0" rot_z="0"
-    effort="1.5" joint_limit_l="-${joint_limit}" joint_limit_u="${joint_limit}" velocity="1.0"
-    damping="10.0" friction="1000.0" />
+    effort="25" joint_limit_l="-${joint_limit}" joint_limit_u="${joint_limit}" velocity="1.5"
+    damping="${damping}" friction="${friction}" />
   <xacro:thigh_link link_name="thigh_link_fr"/>
   <xacro:revolute_joint
@@ -84,6 +86,6 @@
     pos_x="0" pos_y="-0.220" pos_z="0"
     rot_x="0" rot_y="0" rot_z="0"
-    effort="1.5" joint_limit_l="-${joint_limit}" joint_limit_u="${joint_limit}" velocity="1.0"
-    damping="10.0" friction="1000.0" />
+    effort="25" joint_limit_l="-${joint_limit}" joint_limit_u="${joint_limit}" velocity="1.5"
+    damping="${damping}" friction="${friction}" />
   <xacro:leg_link link_name="leg_link_fr"/>
   <!-- ********************** FRONT LEFT LINKS *********************************  -->
@@ -102,6 +104,6 @@
     pos_x="0" pos_y="0" pos_z="0"
     rot_x="0" rot_y="0" rot_z="0"
-    effort="1.5" joint_limit_l="-${joint_limit}" joint_limit_u="${joint_limit}" velocity="1.0"
-    damping="10.0" friction="1000.0" />
+    effort="25" joint_limit_l="-${joint_limit}" joint_limit_u="${joint_limit}" velocity="1.5"
+    damping="${damping}" friction="${friction}" />
   <xacro:thigh_link link_name="thigh_link_fl"/>
   <xacro:revolute_joint
@@ -112,6 +114,6 @@
     pos_x="0" pos_y="-0.220" pos_z="0"
     rot_x="0" rot_y="0" rot_z="0"
-    effort="1.5" joint_limit_l="-${joint_limit}" joint_limit_u="${joint_limit}" velocity="1.0"
-    damping="10.0" friction="1000.0" />
+    effort="25" joint_limit_l="-${joint_limit}" joint_limit_u="${joint_limit}" velocity="1.5"
+    damping="${damping}" friction="${friction}" />
   <xacro:leg_link link_name="leg_link_fl"/>
   <!-- ********************** REAR RIGHT LINKS *********************************  -->
@@ -130,6 +132,6 @@
     pos_x="0" pos_y="0" pos_z="0"
     rot_x="0" rot_y="0" rot_z="0"
-    effort="1.5" joint_limit_l="-${joint_limit}" joint_limit_u="${joint_limit}" velocity="1.0"
-    damping="10.0" friction="1000.0" />
+    effort="25" joint_limit_l="-${joint_limit}" joint_limit_u="${joint_limit}" velocity="1.5"
+    damping="${damping}" friction="${friction}" />
   <xacro:thigh_link link_name="thigh_link_rr"/>
   <xacro:revolute_joint
@@ -140,6 +142,6 @@
     pos_x="0" pos_y="-0.220" pos_z="0"
     rot_x="0" rot_y="0" rot_z="0"
-    effort="1.5" joint_limit_l="-${joint_limit}" joint_limit_u="${joint_limit}" velocity="1.0"
-    damping="10.0" friction="1000.0" />
+    effort="25" joint_limit_l="-${joint_limit}" joint_limit_u="${joint_limit}" velocity="1.5"
+    damping="${damping}" friction="${friction}" />
   <xacro:leg_link link_name="leg_link_rr"/>
   <!-- ********************** REAR LEFT LINKS *********************************  -->
@@ -158,6 +160,6 @@
     pos_x="0" pos_y="0" pos_z="0"
     rot_x="0" rot_y="0" rot_z="0"
-    effort="1.5" joint_limit_l="-${joint_limit}" joint_limit_u="${joint_limit}" velocity="1.0"
-    damping="10.0" friction="1000.0" />
+    effort="25" joint_limit_l="-${joint_limit}" joint_limit_u="${joint_limit}" velocity="1.5"
+    damping="${damping}" friction="${friction}" />
   <xacro:thigh_link link_name="thigh_link_rl"/>
   <xacro:revolute_joint
@@ -168,6 +170,6 @@
     pos_x="0" pos_y="-0.220" pos_z="0"
     rot_x="0" rot_y="0" rot_z="0"
-    effort="1.5" joint_limit_l="-${joint_limit}" joint_limit_u="${joint_limit}" velocity="1.0"
-    damping="10.0" friction="1000.0" />
+    effort="25" joint_limit_l="-${joint_limit}" joint_limit_u="${joint_limit}" velocity="1.5"
+    damping="${damping}" friction="${friction}" />
   <xacro:leg_link link_name="leg_link_rl"/>
 </robot>

File: quad_description/models/quad/quad_gazebo.xacro (robot description, xacro)
@@ -13,4 +13,10 @@
   xmlns:xacro="http://www.ros.org/wiki/xacro">
   <xacro:property name="joint_limit" value="2.09439510239"/>      <!-- 120 degree -->
+  <xacro:property name="kp" value="1000000.0"/>
+  <xacro:property name="kd" value="1.0"/>
+  <xacro:property name="mu1" value="0.15"/>
+  <xacro:property name="mu2" value="0.15"/>
+  <xacro:property name="max_vel" value="0.0"/>
+  <xacro:property name="min_depth" value="0.001"/>
   <gazebo reference="base_link">
     <material>Gazebo/Orange</material>
@@ -27,4 +33,10 @@
   <gazebo reference="leg_link_fr">
     <material>Gazebo/Black</material>
+    <kp>${kp}</kp>
+    <kd>${kd}</kd>
+    <mu1>${mu1}</mu1>
+    <mu2>${mu2}</mu2>
+    <maxVel>${max_vel}</maxVel>
+    <minDepth>${min_depth}</minDepth>
   </gazebo>
   <gazebo reference="hip_link_fl">
@@ -35,4 +47,10 @@
   </gazebo>
   <gazebo reference="leg_link_fl">
+    <kp>${kp}</kp>
+    <kd>${kd}</kd>
+    <mu1>${mu1}</mu1>
+    <mu2>${mu2}</mu2>
+    <maxVel>${max_vel}</maxVel>
+    <minDepth>${min_depth}</minDepth>
     <material>Gazebo/Black</material>
   </gazebo>
@@ -44,4 +62,10 @@
   </gazebo>
   <gazebo reference="leg_link_rr">
+    <kp>${kp}</kp>
+    <kd>${kd}</kd>
+    <mu1>${mu1}</mu1>
+    <mu2>${mu2}</mu2>
+    <maxVel>${max_vel}</maxVel>
+    <minDepth>${min_depth}</minDepth>
     <material>Gazebo/Black</material>
   </gazebo>
@@ -54,4 +78,10 @@
   <gazebo reference="leg_link_rl">
     <material>Gazebo/Black</material>
+    <kp>${kp}</kp>
+    <kd>${kd}</kd>
+    <mu1>${mu1}</mu1>
+    <mu2>${mu2}</mu2>
+    <maxVel>${max_vel}</maxVel>
+    <minDepth>${min_depth}</minDepth>
   </gazebo>
   <gazebo>
