Commit message: fix: added effort-velocity dynamic variable and removed damping-friction

File: quad_description/models/quad/quad.xacro (robot description, xacro)
@@ -5,5 +5,5 @@
 *  Filename:			    quad.xacro
 *  Created:				    22/12/2023
-*  Last Modified:	    31/01/2024
+*  Last Modified:	    01/02/2024
 *  Author:				    Archit Jain
 *
@@ -48,6 +48,6 @@
   <xacro:property name="quad_height" value="1.0"/>
   <xacro:property name="joint_limit" value="2.09439510239"/>      <!-- 120 degree -->
-  <xacro:property name="damping" value="0.5"/>
-  <xacro:property name="friction" value="0.15"/>         <!-- ABS=0.35 -->
+  <xacro:property name="effort" value="25"/>
+  <xacro:property name="velocity" value="1.5"/>
   <!-- ****************** ROBOT BASE FOOTPRINT ***************************  -->
   <!-- Define the center of the main robot chassis projected on the ground -->
@@ -58,5 +58,5 @@
     child_link="base_link"
     pos_x="0" pos_y="0" pos_z="${quad_height}"
-    rot_x="1.571428571" rot_y="0" rot_z="0"/>      <!-- Originally set it to (90 0 0) -->
+    rot_x="1.571428571" rot_y="0" rot_z="0"/>
   <!-- ********************** ROBOT BASELINK *********************************  -->
   <xacro:base_link link_name="base_link"/>
@@ -76,6 +76,5 @@
     pos_x="0" pos_y="0" pos_z="0"
     rot_x="0" rot_y="0" rot_z="0"
-    effort="25" joint_limit_l="-${joint_limit}" joint_limit_u="${joint_limit}" velocity="1.5"
-    damping="${damping}" friction="${friction}" />
+    effort="${effort}" joint_limit_l="-${joint_limit}" joint_limit_u="${joint_limit}" velocity="${velocity}" />
   <xacro:thigh_link link_name="thigh_link_fr"/>
   <xacro:revolute_joint
@@ -86,6 +85,5 @@
     pos_x="0" pos_y="-0.220" pos_z="0"
     rot_x="0" rot_y="0" rot_z="0"
-    effort="25" joint_limit_l="-${joint_limit}" joint_limit_u="${joint_limit}" velocity="1.5"
-    damping="${damping}" friction="${friction}" />
+    effort="${effort}" joint_limit_l="-${joint_limit}" joint_limit_u="${joint_limit}" velocity="${velocity}" />
   <xacro:leg_link link_name="leg_link_fr"/>
   <!-- ********************** FRONT LEFT LINKS *********************************  -->
@@ -104,6 +102,5 @@
     pos_x="0" pos_y="0" pos_z="0"
     rot_x="0" rot_y="0" rot_z="0"
-    effort="25" joint_limit_l="-${joint_limit}" joint_limit_u="${joint_limit}" velocity="1.5"
-    damping="${damping}" friction="${friction}" />
+    effort="${effort}" joint_limit_l="-${joint_limit}" joint_limit_u="${joint_limit}" velocity="${velocity}" />
   <xacro:thigh_link link_name="thigh_link_fl"/>
   <xacro:revolute_joint
@@ -114,6 +111,5 @@
     pos_x="0" pos_y="-0.220" pos_z="0"
     rot_x="0" rot_y="0" rot_z="0"
-    effort="25" joint_limit_l="-${joint_limit}" joint_limit_u="${joint_limit}" velocity="1.5"
-    damping="${damping}" friction="${friction}" />
+    effort="${effort}" joint_limit_l="-${joint_limit}" joint_limit_u="${joint_limit}" velocity="${velocity}" />
   <xacro:leg_link link_name="leg_link_fl"/>
   <!-- ********************** REAR RIGHT LINKS *********************************  -->
@@ -132,6 +128,5 @@
     pos_x="0" pos_y="0" pos_z="0"
     rot_x="0" rot_y="0" rot_z="0"
-    effort="25" joint_limit_l="-${joint_limit}" joint_limit_u="${joint_limit}" velocity="1.5"
-    damping="${damping}" friction="${friction}" />
+    effort="${effort}" joint_limit_l="-${joint_limit}" joint_limit_u="${joint_limit}" velocity="${velocity}" />
   <xacro:thigh_link link_name="thigh_link_rr"/>
   <xacro:revolute_joint
@@ -142,6 +137,5 @@
     pos_x="0" pos_y="-0.220" pos_z="0"
     rot_x="0" rot_y="0" rot_z="0"
-    effort="25" joint_limit_l="-${joint_limit}" joint_limit_u="${joint_limit}" velocity="1.5"
-    damping="${damping}" friction="${friction}" />
+    effort="${effort}" joint_limit_l="-${joint_limit}" joint_limit_u="${joint_limit}" velocity="${velocity}" />
   <xacro:leg_link link_name="leg_link_rr"/>
   <!-- ********************** REAR LEFT LINKS *********************************  -->
@@ -160,6 +154,5 @@
     pos_x="0" pos_y="0" pos_z="0"
     rot_x="0" rot_y="0" rot_z="0"
-    effort="25" joint_limit_l="-${joint_limit}" joint_limit_u="${joint_limit}" velocity="1.5"
-    damping="${damping}" friction="${friction}" />
+    effort="${effort}" joint_limit_l="-${joint_limit}" joint_limit_u="${joint_limit}" velocity="${velocity}" />
   <xacro:thigh_link link_name="thigh_link_rl"/>
   <xacro:revolute_joint
@@ -170,6 +163,5 @@
     pos_x="0" pos_y="-0.220" pos_z="0"
     rot_x="0" rot_y="0" rot_z="0"
-    effort="25" joint_limit_l="-${joint_limit}" joint_limit_u="${joint_limit}" velocity="1.5"
-    damping="${damping}" friction="${friction}" />
+    effort="${effort}" joint_limit_l="-${joint_limit}" joint_limit_u="${joint_limit}" velocity="${velocity}" />
   <xacro:leg_link link_name="leg_link_rl"/>
 </robot>

File: quad_description/models/quad/quad_macros.xacro (robot description, xacro)
@@ -5,5 +5,5 @@
 *  Filename:			    quad_macros.xacro
 *  Created:				    29/01/2024
-*  Last Modified:	    29/01/2024
+*  Last Modified:	    01/02/2024
 *  Author:				    Archit Jain
 *
@@ -38,5 +38,5 @@
     </joint>
   </xacro:macro>
-  <xacro:macro name="revolute_joint" params="joint_name parent_link child_link pos_x pos_y pos_z rot_x rot_y rot_z axis_x axis_y axis_z joint_limit_u joint_limit_l effort velocity damping friction">
+  <xacro:macro name="revolute_joint" params="joint_name parent_link child_link pos_x pos_y pos_z rot_x rot_y rot_z axis_x axis_y axis_z joint_limit_u joint_limit_l effort velocity">
     <joint name="${joint_name}" type="revolute">
       <origin xyz="${pos_x} ${pos_y} ${pos_z}" rpy="${rot_x} ${rot_y} ${rot_z}"/>
@@ -45,5 +45,4 @@
       <axis xyz="${axis_x} ${axis_y} ${axis_z}" />
       <limit effort="${effort}" lower="${joint_limit_l}" upper="${joint_limit_u}" velocity="${velocity}"/>
-      <dynamics damping="${damping}" friction="${friction}" />
     </joint>
   </xacro:macro>
